Commit message: first working version:mapping to zeno joints

File: urdf/pi_robot/pi_arm.urdf.xacro (robot description, xacro)
@@ -1,5 +1,5 @@
 <?xml version="1.0"?>
 <robot name="arm" xmlns:xacro="http://ros.org/wiki/xacro">
-  <xacro:include filename="$(find rbx2_description)/urdf/pi_robot/dynamixel_arm_hardware.xacro" />
+  <xacro:include filename="$(find pi_tracker)/urdf/pi_robot/dynamixel_arm_hardware.xacro" />
   <macro name="arm" params="side reflect parent color *origin">
     <link name="${side}_arm_base_link" />

File: urdf/pi_robot/pi_gripper.urdf.xacro (robot description, xacro)
@@ -27,5 +27,5 @@
         <origin xyz="0 0 0" rpy="0 0 0" />
         <geometry>
-          <mesh filename="package://rbx2_description/meshes/F2.stl" scale="${DYNAMIXEL_MESH_SCALE} ${DYNAMIXEL_MESH_SCALE} ${DYNAMIXEL_MESH_SCALE}"/>
+          <mesh filename="package://pi_tracker/meshes/F2.stl" scale="${DYNAMIXEL_MESH_SCALE} ${DYNAMIXEL_MESH_SCALE} ${DYNAMIXEL_MESH_SCALE}"/>
         </geometry>
         <material name="${color}"/>

File: urdf/pi_robot/pi_pan_tilt_head.urdf.xacro (robot description, xacro)
@@ -5,6 +5,6 @@
   <property name="camera_offset_z" value="0.0615" />
   <property name="camera_mesh_scale" value="1.0" />
-  <xacro:include filename="$(find rbx2_description)/urdf/pi_robot/dynamixel_head_hardware.xacro" />
-  <xacro:include filename="$(find rbx2_description)/urdf/pi_robot/kinect.urdf.xacro" />
+  <xacro:include filename="$(find pi_tracker)/urdf/pi_robot/dynamixel_head_hardware.xacro" />
+  <xacro:include filename="$(find pi_tracker)/urdf/pi_robot/kinect.urdf.xacro" />
   <macro name="head" params="parent name color *origin">
     <!-- head base joint -->

File: urdf/pi_robot/pi_robot_with_two_arms.xacro (robot description, xacro)
@@ -12,10 +12,11 @@
    <property name="arm_offset_z" value="0.70" />
    <!-- The following include files set up definitions of parts of the robot body -->
-   <xacro:include filename="$(find rbx2_description)/urdf/materials.urdf.xacro" />
-   <xacro:include filename="$(find rbx2_description)/urdf/pi_robot/pi_base.urdf.xacro" />
-   <xacro:include filename="$(find rbx2_description)/urdf/pi_robot/pi_torso.urdf.xacro" />
-   <xacro:include filename="$(find rbx2_description)/urdf/pi_robot/pi_pan_tilt_head.urdf.xacro" />
-   <xacro:include filename="$(find rbx2_description)/urdf/pi_robot/pi_arm.urdf.xacro" />
-   <xacro:include filename="$(find rbx2_description)/urdf/pi_robot/pi_gripper.urdf.xacro" />
+   <xacro:include filename="$(find pi_tracker)/urdf/pi_robot/pi_base.urdf.xacro" />
+   <xacro:include filename="$(find pi_tracker)/urdf/pi_robot/pi_torso.urdf.xacro" />
+   <xacro:include filename="$(find pi_tracker)/urdf/pi_robot/pi_pan_tilt_head.urdf.xacro" />
+   <xacro:include filename="$(find pi_tracker)/urdf/pi_robot/pi_arm.urdf.xacro" />
+   <!--
+   <xacro:include filename="$(find pi_tracker)/urdf/pi_robot/pi_gripper.urdf.xacro" />
+   -->
    <!-- Now we can start using the macros included above to define the actual robot -->
    <!-- Start with the base and wheels -->
